File: Julelys V2.kicad_sch (KiCad schematic)
At the start: 16 parts, among them U2 74HC4051

Commit message: Update to V2.1
Parts:
- added D4: 1N5819HW-7-F, Diode_SMD:D_SOD-123, symbol Device:D
Connections:
- net +5V: now also D4.1 (K); no longer V_IN1.2 (Pin_2)
- new net: D4.2 (A), V_IN1.2 (Pin_2)
Other:
- moved on the sheet: CH1, CH2, CH3, CH4, CH5, CH6, CH7, CH8, V_IN1

Commit message: version 3
Parts:
- removed CH1, CH2, CH3, CH4, CH5, CH6, CH7, CH8: Screw_Terminal_01x03, TerminalBlock:TerminalBlock_Altech_AK300-3_P5.00mm, symbol Connector:Screw_Terminal_01x03
- removed D4: 1N5819HW-7-F, Diode_SMD:D_SOD-123, symbol Device:D
- added C8: 100nf, Resistor_SMD:R_0603_1608Metric, symbol Device:C
- added D6: SS34-E3_57T, Diode_SMD:DIOM7959X262N, symbol Diode:SS34-E3_57T
- added J10, J11, J4, J5, J6, J7, J8, J9: B3B-XH-A, Connector:JST_B3B-XH-A, symbol Connector:B3B-XH-A
- added R6: 10K, Resistor_SMD:R_0603_1608Metric, symbol Device:R
- R1, R2, R3: footprint Resistor_SMD:R_0805_2012Metric -> Resistor_SMD:R_0603_1608Metric
Connections:
- net +5V: now also C8.2, D6.C, J10.3, J11.3, J4.3, J5.3, J6.3, J7.3, J8.3, J9.3
- net GND: now also U2.7 (VEE), C8.1, J10.1, J11.1, J4.1, J5.1, J6.1, J7.1, J8.1, J9.1, R6.2
- net at U2.5 (A5): now also J9.2
- net at U2.2 (A6): now also J10.2
- net at U2.1 (A4): now also J8.2
- net at U2.13 (A0): now also J4.2
- net at V_IN1.2 (Pin_2): now also D6.A
- net at U2.12 (A3): now also J7.2
- net at U2.14 (A1): now also J5.2
- net at U2.15 (A2): now also J6.2
- net at U2.4 (A7): now also J11.2
- net at U2.6 (~{E}): now also R6.1
- no-connect marks 2 -> 0

Commit message: Update to v3.1
Parts:
- added R14, R15, R16, R17, R18, R19, R20, R21: 330, Resistor_SMD:R_0603_1608Metric, symbol Device:R
- added U6, U7, U8, U9: 74AHCT1G125, Package_TO_SOT_SMD:SOT-353_SC-70-5, symbol 74xGxx:74AHCT1G125
Connections:
- net +5V: now also U6.5 (VCC), U7.5 (VCC), U8.5 (VCC), U9.5 (VCC)
- net A0: now also U7.2; no longer U2.11 (S0)
- net A1: now also U8.2; no longer U2.10 (S1)
- net A2: now also U9.2; no longer U2.9 (S2)
- net GND: now also U6.1, U6.3 (GND), U7.1, U7.3 (GND), U8.1, U8.3 (GND), U9.1, U9.3 (GND)
- net S1: now also U6.2; no longer U2.3 (A)
- net CH1: now reaches J4.2
- net CH1: now also R14.2; no longer U2.13 (A0)
- net CH5: now reaches J8.2
- net CH5: now also R18.2; no longer U2.1 (A4)
- net CH4: now reaches J7.2
- net CH4: now also R17.2; no longer U2.12 (A3)
- net CH2: now reaches J5.2
- net CH2: now also R15.2; no longer U2.14 (A1)
- net CH3: now reaches J6.2
- net CH3: now also R16.2; no longer U2.15 (A2)
- net CH7: now reaches J10.2
- net CH7: now also R20.2; no longer U2.2 (A6)
- net CH8: now reaches J11.2
- net CH8: now also R21.2; no longer U2.4 (A7)
- net CH6: now reaches J9.2
- net CH6: now also R19.2; no longer U2.5 (A5)
- new net AS0: U2.11 (S0), U7.4
- new net AS1: U2.10 (S1), U8.4
- new net AS2: U2.9 (S2), U9.4
- new net Data: U2.3 (A), U6.4
- new net MCH1: R14.1, U2.13 (A0)
- new net MCH2: R15.1, U2.14 (A1)
- new net MCH3: R16.1, U2.15 (A2)
- new net MCH4: R17.1, U2.12 (A3)
- new net MCH5: R18.1, U2.1 (A4)
- new net MCH6: R19.1, U2.5 (A5)
- new net MCH7: R20.1, U2.2 (A6)
- new net MCH8: R21.1, U2.4 (A7)
Other:
- moved on the sheet: C8, D1, D2, D3, D6, J10, J11, J4, J5, J6, J7, J8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
