File: Julelys.kicad_sch (KiCad schematic)
At the start: 31 parts, among them J10 B3B-XH-A, J11 B3B-XH-A, J4 B3B-XH-A, J5 B3B-XH-A, J6 B3B-XH-A, J7 B3B-XH-A, J8 B3B-XH-A, J9 B3B-XH-A, U2 74HC4051, U6 74AHCT1G125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

Commit message: Begin next step
Parts:
- removed D6: SS34-E3_57T, Diode_SMD:DIOM7959X262N, symbol Diode:SS34-E3_57T
- added TP1: 5V, TestPoint:TestPoint_Pad_1.0x1.0mm, symbol Connector:TestPoint
- added TP2: GND, TestPoint:TestPoint_Pad_1.0x1.0mm, symbol Connector:TestPoint
- added V_IN2: 5V, TerminalBlock:TerminalBlock_Altech_AK300-2_P5.00mm, symbol Connector:Screw_Terminal_01x02
Connections:
- net +5V: now also V_IN1.2 (Pin_2), TP1.1, V_IN2.2 (Pin_2)
- net GND: now also TP2.1, V_IN2.1 (Pin_1)
