File: Julelys.kicad_sch (KiCad schematic)
At the start: 33 parts, among them J10 B3B-XH-A, J11 B3B-XH-A, J4 B3B-XH-A, J5 B3B-XH-A, J6 B3B-XH-A, J7 B3B-XH-A, J8 B3B-XH-A, J9 B3B-XH-A, U2 74HC4051, U6 74AHCT1G125, U7 74AHCT1G125, U8 74AHCT1G125, U9 74AHCT1G125

Commit message: Rework v4 schematic for Raspberry Pi 4/5 HAT
- Remap J1 to the Raspberry Pi 40-pin pinout (was still Orange Pi pin
  numbers: Pi 3V3 on MISO, GND on ESP32 RX)
- Fix auto-reset: U4 collectors drove EN and IO9 the wrong way round
- Let the Pi flash the ESP32: UART via 74LVC1G08 AND gate (U10) shared
  with the CP2102N, EN/BOOT on GPIO5/6 through 1k; add IO9 pull-up
- Power the Pi straight from +5V, drop the SS34 diode (D6)
- Add fan control: AO3400A low-side switch on GPIO18, tach on GPIO24
- Move mux LEDs D1-D3 off strapping pin GPIO8 to the 5V select lines
- Add 3V3 power LED and test points TP8-TP33
- Document v4 in CLAUDE.md

Co-Authored-By: Claude Opus 5.5 <noreply@anthropic.com>
Parts:
- added TP22: DATA, TestPoint:TestPoint_Pad_1.0x1.0mm, symbol Connector:TestPoint
- added TP23: AS0, TestPoint:TestPoint_Pad_1.0x1.0mm, symbol Connector:TestPoint
- added TP24: AS1, TestPoint:TestPoint_Pad_1.0x1.0mm, symbol Connector:TestPoint
- added TP25: AS2, TestPoint:TestPoint_Pad_1.0x1.0mm, symbol Connector:TestPoint
- added TP26: CH1, TestPoint:TestPoint_Pad_1.0x1.0mm, symbol Connector:TestPoint
- added TP27: CH2, TestPoint:TestPoint_Pad_1.0x1.0mm, symbol Connector:TestPoint
- added TP28: CH3, TestPoint:TestPoint_Pad_1.0x1.0mm, symbol Connector:TestPoint
- added TP29: CH4, TestPoint:TestPoint_Pad_1.0x1.0mm, symbol Connector:TestPoint
- added TP30: CH5, TestPoint:TestPoint_Pad_1.0x1.0mm, symbol Connector:TestPoint
- added TP31: CH6, TestPoint:TestPoint_Pad_1.0x1.0mm, symbol Connector:TestPoint
- added TP32: CH7, TestPoint:TestPoint_Pad_1.0x1.0mm, symbol Connector:TestPoint
- added TP33: CH8, TestPoint:TestPoint_Pad_1.0x1.0mm, symbol Connector:TestPoint
- R1, R2, R3: value 270 -> 1K
Connections:
- net A0: no longer D1.2 (A)
- net A1: no longer D2.2 (A)
- net A2: no longer D3.2 (A)
- net AS0: now also D1.2 (A), TP23.1
- net AS1: now also D2.2 (A), TP24.1
- net AS2: now also D3.2 (A), TP25.1
- net CH1: now also TP26.1
- net CH2: now also TP27.1
- net CH3: now also TP28.1
- net CH4: now also TP29.1
- net CH5: now also TP30.1
- net CH6: now also TP31.1
- net CH7: now also TP32.1
- net CH8: now also TP33.1
- net Data: now also TP22.1

Commit message: Add 3D models for all parts, turn screw terminals to face the board edge
- Point library parts at KiCad 10 STEP models; copy the HRO USB-C and
  ESP32-C3 models into 3D/ so the project is self-contained
- Add models for U2 (SOIC-16) and U5 (CP2102N); use the KiCad TL3305A
  model instead of a file in Downloads
- Rotate V_IN1/V_IN2 so the 45-degree wire entry faces the left edge;
  mirror the symbols (pin 1 = +5V, pin 2 = GND) so the power tracks stay
- Reroute TXD and PI_TX segments that came too close to the new pads
- Document Pi 5 Active Cooler mounting (GPIO extension, taller standoffs)

Co-Authored-By: Claude Opus 5.5 <noreply@anthropic.com>
Connections:
- net +5V: now also V_IN1.1 (Pin_1), V_IN2.1 (Pin_1); no longer V_IN1.2 (Pin_2), V_IN2.2 (Pin_2)
- net GND: now also V_IN1.2 (Pin_2), V_IN2.2 (Pin_2); no longer V_IN1.1 (Pin_1), V_IN2.1 (Pin_1)
Changed lines of the file:
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@@
     )
   )
-  (symbol (lib_id "Connector:Screw_Terminal_01x02") (at 157.48 58.42 0) (unit 1)
+  (symbol (lib_id "Connector:Screw_Terminal_01x02") (at 157.48 60.96 0) (mirror x) (unit 1)
     (in_bom yes) (on_board yes) (dnp no) (fields_autoplaced)
     (property "Reference" "V_IN2" (at 160.02 58.42 0)
@@
     )
   )
-  (symbol (lib_id "Connector:Screw_Terminal_01x02") (at 157.48 67.31 0) (unit 1)
+  (symbol (lib_id "Connector:Screw_Terminal_01x02") (at 157.48 69.85 0) (mirror x) (unit 1)
     (in_bom yes) (on_board yes) (dnp no) (fields_autoplaced)
     (property "Reference" "V_IN1" (at 160.02 67.31 0)

Commit message: Apply schematic review fixes, add JLCPCB rules, prepare for manual layout
Schematic (from a Codex review):
- R35 10k pull-up on GPIO2 (strapping pin; Pi MISO has a default pull-down)
- R36 10k pull-down on IO7 so the LEDs stay dark while the ESP32 boots
- C5 22uF for AMS1117 output stability, C7 1nF on GPIO9
- C18-C21 100nF decoupling for the level shifters U6-U9

Board:
- New parts parked outside the outline for manual placement
- Silkscreen scaled to JLCPCB's 1.0 mm minimum; back pinout table rebuilt
- C5/C7 values synced

Rules:
- JLCPCB 4-layer limits in Julelys.kicad_pro and new Julelys.kicad_dru

Co-Authored-By: Claude Opus 5.5 <noreply@anthropic.com>
Parts:
- added C18, C19, C20, C21: 100nF, Capacitor_SMD:C_0603_1608Metric, symbol Device:C
Connections:
- net +5V: now also C18.1, C19.1, C20.1, C21.1
- net GND: now also C18.2, C19.2, C20.2, C21.2
Other:
- note added: "Decoupling for U6-U9 (place at VCC pin)"

Commit message: Test board schematic: bare ESP32-C3FH4, native USB, noise fixes
A - bare chip (docs/esp32-c3-chip-design.md):
- ESP32-C3FH4 (4 MB in-package flash) replaces the WROOM-02 module
- Espressif reference core: VDD3P3 2.0 nH filter + 1 uF, VDDA 1 uF + 10 nF,
  RTC/CPU 100 nF, VDD_SPI 1 uF, 40 MHz crystal with 24 nH series and 22 pF
- RF: CLC match at the chip, pi footprint with 6.8 nH at a Walsin
  RFANT3216120A5T chip antenna (shunts DNP for tuning)
- 499 ohm on U0TXD

B - native USB:
- USB-C D+/D- via ESD and 22 ohm to GPIO19/18 (USB Serial/JTAG);
  D+ pull-up footprint DNP
- CP2102N, DTR/RTS auto-reset and the UART AND gate removed; J1 pin 8
  drives ESP32 RX directly (R27 pull-up)

Noise fixes (docs/noise-analysis-v4.md):
- 10k pull-downs and SRV05-4 TVS arrays on CH1-CH8
- SMBJ5.0A TVS on +5V, 100 uF at J1, 3 x 100 nF spread on +5V

ERC: 0 errors. Board layout not updated yet.

Co-Authored-By: Claude Opus 5.5 <noreply@anthropic.com>
Parts:
- added C37, C38, C39: 100nF, Capacitor_SMD:C_0402_1005Metric, symbol Device:C
- added D10: SMBJ5.0A, Diode_SMD:D_SMB, symbol Device:D_TVS
- added R43, R44, R45, R46, R47, R48, R49, R50: 10K, Resistor_SMD:R_0402_1005Metric, symbol Device:R
- added U11, U12: SRV05-4, Package_TO_SOT_SMD:SOT-23-6, symbol Power_Protection:SRV05-4
Connections:
- net +5V: now also C37.1, C38.1, C39.1, D10.1 (A1), U11.5 (VP), U12.5 (VP)
- net CH1: now also R43.1, U11.1 (IO1)
- net CH2: now also R44.1, U11.3 (IO2)
- net CH3: now also R45.1, U11.4 (IO3)
- net CH4: now also R46.1, U11.6 (IO4)
- net CH5: now also R47.1, U12.1 (IO1)
- net CH6: now also R48.1, U12.3 (IO2)
- net CH7: now also R49.1, U12.4 (IO3)
- net CH8: now also R50.1, U12.6 (IO4)
- net GND: now also C37.2, C38.2, C39.2, D10.2 (A2), R43.2, R44.2, R45.2, R46.2, R47.2, R48.2, R49.2, R50.2, U11.2 (VN), U12.2 (VN)
Other:
- note added: "Noise fixes (docs/noise-analysis-v4.md): R43-R50 pull-downs keep idle LED inputs low, U11/U12 TVS on the LED outputs, D10 TVS on +5V, C37-C39 spread +5V/GND decoupling."

Commit message: Test board: read 8 analog sensors through the LED JST outputs
- U6 /OE now on IO1 (R51 10k pull-down keeps it on at boot); IO1 high
  tri-states the LED data shifter.
- /Data -> R52 15k -> IO0 (ADC1_CH0) -> R53 10k + C40 10nF to GND, so the
  mux can route any JST data pin back to the ADC (0-5 V -> 0-2 V).
- Placed and routed; references re-placed. 0 DRC errors, 0 unconnected,
  no silkscreen warnings, ERC unchanged.
- docs/sensor-input.md: how it works, read sequence, limits.

Co-Authored-By: Claude Opus 5.5 <noreply@anthropic.com>
Parts:
- added C40: 10nF, Capacitor_SMD:C_0402_1005Metric, symbol Device:C
- added R51, R53: 10k, Resistor_SMD:R_0402_1005Metric, symbol Device:R
- added R52: 15k, Resistor_SMD:R_0402_1005Metric, symbol Device:R
Connections:
- net Data: now also R52.1
- net GND: now also C40.2, R51.2, R53.2; no longer U6.1
- new net IO0: C40.1, R52.2, R53.1
- new net IO1: R51.1, U6.1
Other:
- note added: "Sensor read-back on J4-J11: IO1 high tri-states U6, A0-A2 select the channel, IO0 (ADC1_CH0) reads it through R52/R53 (0-5 V -> 0-2 V). R51 keeps U6 on at boot."
Changed lines of the file:
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@@
   (junction (at 44.45 38.1) (diameter 0) (color 0 0 0 0)
   )
-  (junction (at 118.11 67.31) (diameter 0) (color 0 0 0 0)
-  )
   (junction (at 130.81 54.61) (diameter 0) (color 0 0 0 0)
   )
@@
     (stroke (width 0) (type default))
   )
-  (wire (pts (xy 111.76 67.31) (xy 118.11 67.31))
-    (stroke (width 0) (type default))
-  )
   (wire (pts (xy 96.52 101.6) (xy 105.41 101.6))
     (stroke (width 0) (type default))
@@
     (stroke (width 0) (type default))
   )
-  (wire (pts (xy 111.76 59.69) (xy 111.76 67.31))
-    (stroke (width 0) (type default))
-  )
   (label "CH8" (at 144.78 160.02 0) (fields_autoplaced)
     (effects (font (size 1.27 1.27)) (justify left bottom))
@@
     (effects (font (size 1.27 1.27)) (justify left bottom))
   )
+  (wire (pts (xy 111.76 59.69) (xy 111.76 64.77))
+    (stroke (width 0) (type default))
+  )
+  (global_label "IO1" (shape input) (at 111.76 64.77 270) (fields_autoplaced)
+    (effects (font (size 1.27 1.27)) (justify right))
+    (property "Intersheetrefs" "${INTERSHEET_REFS}" (at 111.76 64.77 270)
+      (effects (font (size 1.27 1.27)) (justify right) hide)
+    )
+  )
+  (symbol (lib_id "Device:R") (at 190.5 182.88 0) (unit 1)
+    (in_bom yes) (on_board yes) (dnp no)
+    (property "Reference" "R52" (at 192.532 182.88 90)
+      (effects (font (size 1.27 1.27)))
+    )
+    (property "Value" "15k" (at 190.5 182.88 90)
+      (effects (font (size 1.27 1.27)))
+    )
+    (property "Footprint" "Resistor_SMD:R_0402_1005Metric" (at 188.722 182.88 90)
+      (effects (font (size 1.27 1.27)) hide)
+    )
+    (property "Datasheet" "~" (at 190.5 182.88 0)
+      (effects (font (size 1.27 1.27)) hide)
+    )
+    (pin "1")
+    (pin "2")
+    (instances
+      (project "Julelys"
+        (path "/9ef41b73-8dcb-4021-8930-5b1db22eb182"
+          (reference "R52") (unit 1)
+        )
+      )
+    )
+  )
+  (symbol (lib_id "Device:R") (at 190.5 193.04 0) (unit 1)
+    (in_bom yes) (on_board yes) (dnp no)
+    (property "Reference" "R53" (at 192.532 193.04 90)
+      (effects (font (size 1.27 1.27)))
+    )
+    (property "Value" "10k" (at 190.5 193.04 90)
+      (effects (font (size 1.27 1.27)))
+    )
+    (property "Footprint" "Resistor_SMD:R_0402_1005Metric" (at 188.722 193.04 90)
+      (effects (font (size 1.27 1.27)) hide)
+    )
+    (property "Datasheet" "~" (at 190.5 193.04 0)
+      (effects (font (size 1.27 1.27)) hide)
+    )
+    (pin "1")
+    (pin "2")
+    (instances
+      (project "Julelys"
+        (path "/9ef41b73-8dcb-4021-8930-5b1db22eb182"
+          (reference "R53") (unit 1)
+        )
+      )
+    )
+  )
+  (symbol (lib_id "Device:C") (at 195.58 193.04 0) (unit 1)
+    (in_bom yes) (on_board yes) (dnp no)
+    (property "Reference" "C40" (at 196.215 190.5 0)
+      (effects (font (size 1.27 1.27)) (justify left))
+    )
+    (property "Value" "10nF" (at 196.215 195.58 0)
+      (effects (font (size 1.27 1.27)) (justify left))
+    )
+    (property "Footprint" "Capacitor_SMD:C_0402_1005Metric" (at 196.5452 196.85 0)
+      (effects (font (size 1.27 1.27)) hide)
+    )
+    (property "Datasheet" "~" (at 195.58 193.04 0)
+      (effects (font (size 1.27 1.27)) hide)
+    )
+    (pin "1")
+    (pin "2")
+    (instances
+      (project "Julelys"
+        (path "/9ef41b73-8dcb-4021-8930-5b1db22eb182"
+          (reference "C40") (unit 1)
+        )
+      )
+    )
+  )
+  (symbol (lib_id "Device:R") (at 213.36 193.04 0) (unit 1)
+    (in_bom yes) (on_board yes) (dnp no)
+    (property "Reference" "R51" (at 215.392 193.04 90)
+      (effects (font (size 1.27 1.27)))
+    )
+    (property "Value" "10k" (at 213.36 193.04 90)
+      (effects (font (size 1.27 1.27)))
+    )
+    (property "Footprint" "Resistor_SMD:R_0402_1005Metric" (at 211.582 193.04 90)
+      (effects (font (size 1.27 1.27)) hide)
+    )
+    (property "Datasheet" "~" (at 213.36 193.04 0)
+      (effects (font (size 1.27 1.27)) hide)
+    )
+    (pin "1")
+    (pin "2")
+    (instances
+      (project "Julelys"
+        (path "/9ef41b73-8dcb-4021-8930-5b1db22eb182"
+          (reference "R51") (unit 1)
+        )
+      )
+    )
+  )
+  (wire (pts (xy 190.5 179.07) (xy 190.5 176.53))
+    (stroke (width 0) (type default))
+  )
+  (label "Data" (at 190.5 176.53 90) (fields_autoplaced)
+    (effects (font (size 1.27 1.27)) (justify left bottom))
+  )
+  (wire (pts (xy 190.5 186.69) (xy 190.5 189.23))
+    (stroke (width 0) (type default))
+  )
+  (wire (pts (xy 190.5 189.23) (xy 195.58 189.23))
+    (stroke (width 0) (type default))
+  )
+  (wire (pts (xy 195.58 189.23) (xy 200.66 189.23))
+    (stroke (width 0) (type default))
+  )
+  (global_label "IO0" (shape input) (at 200.66 189.23 0) (fields_autoplaced)
+    (effects (font (size 1.27 1.27)) (justify left))
+    (property "Intersheetrefs" "${INTERSHEET_REFS}" (at 200.66 189.23 0)
+      (effects (font (size 1.27 1.27)) (justify left) hide)
+    )
+  )
+  (junction (at 190.5 189.23) (diameter 0) (color 0 0 0 0)
+  )
+  (junction (at 195.58 189.23) (diameter 0) (color 0 0 0 0)
+  )
+  (wire (pts (xy 190.5 196.85) (xy 190.5 199.39))
+    (stroke (width 0) (type default))
+  )
+  (symbol (lib_id "power:GND") (at 190.5 199.39 0) (unit 1)
+    (in_bom yes) (on_board yes) (dnp no) (fields_autoplaced)
+    (property "Reference" "#PWR0401" (at 190.5 199.39 0)
+      (effects (font (size 1.27 1.27)) hide)
+    )
+    (property "Value" "GND" (at 190.5 203.2 0)
+      (effects (font (size 1.27 1.27)))
+    )
+    (property "Footprint" "" (at 190.5 199.39 0)
+      (effects (font (size 1.27 1.27)) hide)
+    )
+    (property "Datasheet" "" (at 190.5 199.39 0)
+      (effects (font (size 1.27 1.27)) hide)
+    )
+    (pin "1")
+    (instances
+      (project "Julelys"
+        (path "/9ef41b73-8dcb-4021-8930-5b1db22eb182"
+          (reference "#PWR0401") (unit 1)
+        )
+      )
+    )
+  )
+  (wire (pts (xy 195.58 196.85) (xy 195.58 199.39))
+    (stroke (width 0) (type default))
+  )
+  (symbol (lib_id "power:GND") (at 195.58 199.39 0) (unit 1)
+    (in_bom yes) (on_board yes) (dnp no) (fields_autoplaced)
+    (property "Reference" "#PWR0402" (at 195.58 199.39 0)
+      (effects (font (size 1.27 1.27)) hide)
+    )
+    (property "Value" "GND" (at 195.58 203.2 0)
+      (effects (font (size 1.27 1.27)))
+    )
+    (property "Footprint" "" (at 195.58 199.39 0)
+      (effects (font (size 1.27 1.27)) hide)
+    )
+    (property "Datasheet" "" (at 195.58 199.39 0)
+      (effects (font (size 1.27 1.27)) hide)
+    )
+    (pin "1")
+    (instances
+      (project "Julelys"
+        (path "/9ef41b73-8dcb-4021-8930-5b1db22eb182"
+          (reference "#PWR0402") (unit 1)
+        )
+      )
+    )
+  )
+  (wire (pts (xy 213.36 189.23) (xy 213.36 186.69))
+    (stroke (width 0) (type default))
+  )
+  (global_label "IO1" (shape input) (at 213.36 186.69 90) (fields_autoplaced)
+    (effects (font (size 1.27 1.27)) (justify left))
+    (property "Intersheetrefs" "${INTERSHEET_REFS}" (at 213.36 186.69 90)
+      (effects (font (size 1.27 1.27)) (justify left) hide)
+    )
+  )
+  (wire (pts (xy 213.36 196.85) (xy 213.36 199.39))
+    (stroke (width 0) (type default))
+  )
+  (symbol (lib_id "power:GND") (at 213.36 199.39 0) (unit 1)
+    (in_bom yes) (on_board yes) (dnp no) (fields_autoplaced)
+    (property "Reference" "#PWR0403" (at 213.36 199.39 0)
+      (effects (font (size 1.27 1.27)) hide)
+    )
+    (property "Value" "GND" (at 213.36 203.2 0)
+      (effects (font (size 1.27 1.27)))
+    )
+    (property "Footprint" "" (at 213.36 199.39 0)
+      (effects (font (size 1.27 1.27)) hide)
+    )
+    (property "Datasheet" "" (at 213.36 199.39 0)
+      (effects (font (size 1.27 1.27)) hide)
+    )
+    (pin "1")
+    (instances
+      (project "Julelys"
+        (path "/9ef41b73-8dcb-4021-8930-5b1db22eb182"
+          (reference "#PWR0403") (unit 1)
+        )
+      )
+    )
+  )
+  (text "Sensor read-back on J4-J11: IO1 high tri-states U6, A0-A2 select the channel,\nIO0 (ADC1_CH0) reads it through R52/R53 (0-5 V -> 0-2 V). R51 keeps U6 on at boot." (at 180.34 172.72 0)
+    (effects (font (size 1.27 1.27)) (justify left bottom))
+  )
