File: esp32.kicad_sch (KiCad schematic)
At the start: 5 parts, among them U1 ESP32-C3-WROOM-02

Commit message: version 3
Parts:
- C1, C2, C3: footprint Capacitor_SMD:C_0805_2012Metric -> Capacitor_SMD:C_0603_1608Metric
- R4: footprint Resistor_SMD:R_0805_2012Metric -> Resistor_SMD:R_0603_1608Metric
Connections:
- net IO4 is gone; now on net A0: U1.3 (GPIO4/ADC1_CH4)
- net IO5 is gone; now on net A1: U1.4 (GPIO5/ADC2_CH0)
- net A0: no longer U1.5 (GPIO6)
- net A1: no longer U1.6 (GPIO7)
- net IO10 renamed CS
- net U-RX renamed RXD
- net U-TX renamed TXD
- new net CLK: U1.5 (GPIO6)
- new net IO7: U1.6 (GPIO7)

Commit message: Update to v3.1
Parts:
- added R23: 10K, Resistor_SMD:R_0603_1608Metric, symbol Device:R
Connections:
- net IO3 is gone; now on net CLK: U1.15 (GPIO3/ADC1_CH3)
- net +3.3V: now also R23.1
- net A2: now also R23.2
- net CLK: no longer U1.5 (GPIO6)
- new net IO6: U1.5 (GPIO6)

Commit message: Begin next step
Parts:
- added TP4: MOSI, TestPoint:TestPoint_Pad_1.0x1.0mm, symbol Connector:TestPoint
- added TP5: MISO, TestPoint:TestPoint_Pad_1.0x1.0mm, symbol Connector:TestPoint
- added TP6: CLK, TestPoint:TestPoint_Pad_1.0x1.0mm, symbol Connector:TestPoint
- added TP7: CS, TestPoint:TestPoint_Pad_1.0x1.0mm, symbol Connector:TestPoint
Connections:
- net CLK: now also TP6.1
- net CS: now also TP7.1
- net IO2: now also TP5.1
- net IO6: now also TP4.1
Changed lines of the file:
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@@
     (stroke (width 0) (type default))
   )
-  (wire (pts (xy 110.49 102.87) (xy 110.49 109.22))
+  (wire (pts (xy 110.49 102.87) (xy 110.49 105.41))
     (stroke (width 0) (type default))
   )
@@
     (stroke (width 0) (type default))
   )
-  (wire (pts (xy 124.46 124.46) (xy 128.27 124.46))
+  (wire (pts (xy 96.52 124.46) (xy 128.27 124.46))
     (stroke (width 0) (type default))
   )
@@
     (stroke (width 0) (type default))
   )
-  (wire (pts (xy 124.46 119.38) (xy 128.27 119.38))
-    (stroke (width 0) (type default))
-  )
   (wire (pts (xy 166.37 116.84) (xy 184.15 116.84))
     (stroke (width 0) (type default))
@@
     (stroke (width 0) (type default))
   )
-  (wire (pts (xy 124.46 127) (xy 128.27 127))
+  (wire (pts (xy 91.44 127) (xy 128.27 127))
     (stroke (width 0) (type default))
   )
@@
     (stroke (width 0) (type default))
   )
+  (wire (pts (xy 105.41 119.38) (xy 128.27 119.38))
+    (stroke (width 0) (type default))
+  )
+  (wire (pts (xy 101.6 121.92) (xy 128.27 121.92))
+    (stroke (width 0) (type default))
+  )
   (wire (pts (xy 44.45 101.6) (xy 52.07 101.6))
     (stroke (width 0) (type default))
@@
   )
   (wire (pts (xy 144.78 92.71) (xy 144.78 143.51))
-    (stroke (width 0) (type default))
-  )
-  (wire (pts (xy 124.46 121.92) (xy 128.27 121.92))
     (stroke (width 0) (type default))
   )
@@
     (pin "2")
     (instances
-      (project "Julelys V2"
+      (project "Julelys"
         (path "/9ef41b73-8dcb-4021-8930-5b1db22eb182/9665c677-0b50-4f2a-bdc6-f5e1c3cc96ed"
           (reference "C2") (unit 1)
@@
     (pin "13")
     (instances
-      (project "Julelys V2"
+      (project "Julelys"
         (path "/9ef41b73-8dcb-4021-8930-5b1db22eb182/9665c677-0b50-4f2a-bdc6-f5e1c3cc96ed"
           (reference "U1") (unit 1)
@@
     (pin "1")
     (instances
-      (project "Julelys V2"
+      (project "Julelys"
         (path "/9ef41b73-8dcb-4021-8930-5b1db22eb182/9665c677-0b50-4f2a-bdc6-f5e1c3cc96ed"
           (reference "#PWR03") (unit 1)
@@
     (pin "2")
     (instances
-      (project "Julelys V2"
+      (project "Julelys"
         (path "/9ef41b73-8dcb-4021-8930-5b1db22eb182/9665c677-0b50-4f2a-bdc6-f5e1c3cc96ed"
           (reference "C1") (unit 1)
@@
     )
   )
-  (symbol (lib_id "power:GND") (at 110.49 109.22 0) (unit 1)
-    (in_bom yes) (on_board yes) (dnp no) (fields_autoplaced)
-    (property "Reference" "#PWR04" (at 110.49 115.57 0)
-      (effects (font (size 1.27 1.27)) hide)
-    )
-    (property "Value" "GND" (at 110.49 114.3 0)
-      (effects (font (size 1.27 1.27)))
-    )
-    (property "Footprint" "" (at 110.49 109.22 0)
-      (effects (font (size 1.27 1.27)) hide)
-    )
-    (property "Datasheet" "" (at 110.49 109.22 0)
-      (effects (font (size 1.27 1.27)) hide)
-    )
-    (pin "1")
-    (instances
-      (project "Julelys V2"
+  (symbol (lib_id "power:GND") (at 110.49 105.41 0) (unit 1)
+    (in_bom yes) (on_board yes) (dnp no) (fields_autoplaced)
+    (property "Reference" "#PWR04" (at 110.49 111.76 0)
+      (effects (font (size 1.27 1.27)) hide)
+    )
+    (property "Value" "GND" (at 110.49 110.49 0)
+      (effects (font (size 1.27 1.27)))
+    )
+    (property "Footprint" "" (at 110.49 105.41 0)
+      (effects (font (size 1.27 1.27)) hide)
+    )
+    (property "Datasheet" "" (at 110.49 105.41 0)
+      (effects (font (size 1.27 1.27)) hide)
+    )
+    (pin "1")
+    (instances
+      (project "Julelys"
         (path "/9ef41b73-8dcb-4021-8930-5b1db22eb182/9665c677-0b50-4f2a-bdc6-f5e1c3cc96ed"
           (reference "#PWR04") (unit 1)
@@
     (pin "2")
     (instances
-      (project "Julelys V2"
+      (project "Julelys"
         (path "/9ef41b73-8dcb-4021-8930-5b1db22eb182/9665c677-0b50-4f2a-bdc6-f5e1c3cc96ed"
           (reference "R4") (unit 1)
@@
     (pin "1")
     (instances
-      (project "Julelys V2"
+      (project "Julelys"
         (path "/9ef41b73-8dcb-4021-8930-5b1db22eb182/9665c677-0b50-4f2a-bdc6-f5e1c3cc96ed"
           (reference "#PWR06") (unit 1)
@@
     (pin "1")
     (instances
-      (project "Julelys V2"
+      (project "Julelys"
         (path "/9ef41b73-8dcb-4021-8930-5b1db22eb182/9665c677-0b50-4f2a-bdc6-f5e1c3cc96ed"
           (reference "#PWR05") (unit 1)
@@
     )
   )
+  (symbol (lib_id "Connector:TestPoint") (at 105.41 119.38 0) (unit 1)
+    (in_bom yes) (on_board yes) (dnp no)
+    (property "Reference" "TP4" (at 105.41 113.03 0)
+      (effects (font (size 1.27 1.27)))
+    )
+    (property "Value" "MOSI" (at 109.22 115.57 0)
+      (effects (font (size 1.27 1.27)))
+    )
+    (property "Footprint" "TestPoint:TestPoint_Pad_1.0x1.0mm" (at 110.49 119.38 0)
+      (effects (font (size 1.27 1.27)) hide)
+    )
+    (property "Datasheet" "~" (at 110.49 119.38 0)
+      (effects (font (size 1.27 1.27)) hide)
+    )
+    (pin "1")
+    (instances
+      (project "Julelys"
+        (path "/9ef41b73-8dcb-4021-8930-5b1db22eb182/9665c677-0b50-4f2a-bdc6-f5e1c3cc96ed"
+          (reference "TP4") (unit 1)
+        )
+      )
+    )
+  )
+  (symbol (lib_id "Connector:TestPoint") (at 101.6 121.92 0) (unit 1)
+    (in_bom yes) (on_board yes) (dnp no)
+    (property "Reference" "TP5" (at 99.06 115.57 0)
+      (effects (font (size 1.27 1.27)))
+    )
+    (property "Value" "MISO" (at 99.06 118.11 0)
+      (effects (font (size 1.27 1.27)))
+    )
+    (property "Footprint" "TestPoint:TestPoint_Pad_1.0x1.0mm" (at 106.68 121.92 0)
+      (effects (font (size 1.27 1.27)) hide)
+    )
+    (property "Datasheet" "~" (at 106.68 121.92 0)
+      (effects (font (size 1.27 1.27)) hide)
+    )
+    (pin "1")
+    (instances
+      (project "Julelys"
+        (path "/9ef41b73-8dcb-4021-8930-5b1db22eb182/9665c677-0b50-4f2a-bdc6-f5e1c3cc96ed"
+          (reference "TP5") (unit 1)
+        )
+      )
+    )
+  )
+  (symbol (lib_id "Connector:TestPoint") (at 96.52 124.46 0) (unit 1)
+    (in_bom yes) (on_board yes) (dnp no)
+    (property "Reference" "TP6" (at 93.98 118.11 0)
+      (effects (font (size 1.27 1.27)))
+    )
+    (property "Value" "CLK" (at 93.98 120.65 0)
+      (effects (font (size 1.27 1.27)))
+    )
+    (property "Footprint" "TestPoint:TestPoint_Pad_1.0x1.0mm" (at 101.6 124.46 0)
+      (effects (font (size 1.27 1.27)) hide)
+    )
+    (property "Datasheet" "~" (at 101.6 124.46 0)
+      (effects (font (size 1.27 1.27)) hide)
+    )
+    (pin "1")
+    (instances
+      (project "Julelys"
+        (path "/9ef41b73-8dcb-4021-8930-5b1db22eb182/9665c677-0b50-4f2a-bdc6-f5e1c3cc96ed"
+          (reference "TP6") (unit 1)
+        )
+      )
+    )
+  )
+  (symbol (lib_id "Connector:TestPoint") (at 91.44 127 0) (unit 1)
+    (in_bom yes) (on_board yes) (dnp no)
+    (property "Reference" "TP7" (at 88.9 120.65 0)
+      (effects (font (size 1.27 1.27)))
+    )
+    (property "Value" "CS" (at 88.9 123.19 0)
+      (effects (font (size 1.27 1.27)))
+    )
+    (property "Footprint" "TestPoint:TestPoint_Pad_1.0x1.0mm" (at 96.52 127 0)
+      (effects (font (size 1.27 1.27)) hide)
+    )
+    (property "Datasheet" "~" (at 96.52 127 0)
+      (effects (font (size 1.27 1.27)) hide)
+    )
+    (pin "1")
+    (instances
+      (project "Julelys"
+        (path "/9ef41b73-8dcb-4021-8930-5b1db22eb182/9665c677-0b50-4f2a-bdc6-f5e1c3cc96ed"
+          (reference "TP7") (unit 1)
+        )
+      )
+    )
+  )
   (symbol (lib_id "Device:C") (at 73.66 43.18 0) (unit 1)
     (in_bom yes) (on_board yes) (dnp no) (fields_autoplaced)
@@
     (pin "1")
     (instances
-      (project "Julelys V2"
+      (project "Julelys"
         (path "/9ef41b73-8dcb-4021-8930-5b1db22eb182/9665c677-0b50-4f2a-bdc6-f5e1c3cc96ed"
           (reference "C3") (unit 1)
@@
     (pin "2")
     (instances
-      (project "Julelys V2"
+      (project "Julelys"
         (path "/9ef41b73-8dcb-4021-8930-5b1db22eb182/9665c677-0b50-4f2a-bdc6-f5e1c3cc96ed"
           (reference "R23") (unit 1)
