File: Julelys.kicad_pcb (KiCad board)
At the start: 4 copper layers, 60 x 53 mm, 75 parts, among them J1 Conn_02x13_Top_Bottom, J10 B3B-XH-A, J11 B3B-XH-A, J12 Conn_01x03_Pin, J2 Conn_01x13, J3 Conn_02x06_Odd_Even, J4 B3B-XH-A, J5 B3B-XH-A, J6 B3B-XH-A, J7 B3B-XH-A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

Commit message: more to next step
Parts:
- added C15: 470uF, Capacitor_SMD:CP_Elec_8x10, F.Cu at (111.8, 48.8)
- added C16: 100nF, Capacitor_SMD:C_0603_1608Metric, F.Cu at (118.7, 54.9)
- added TP1: 5V, TestPoint:TestPoint_Pad_1.0x1.0mm, F.Cu at (133.5, 40.4)
- added TP2: GND, TestPoint:TestPoint_Pad_1.0x1.0mm, F.Cu at (119.5, 32.4)
- added TP3: 3.3V, TestPoint:TestPoint_Pad_1.0x1.0mm, F.Cu at (112.1, 66.3)
- added TP4: MOSI, TestPoint:TestPoint_Pad_1.0x1.0mm, F.Cu at (124.2, 45.4)
- added TP5: MISO, TestPoint:TestPoint_Pad_1.0x1.0mm, F.Cu at (124.2, 48.4)
- added TP6: CLK, TestPoint:TestPoint_Pad_1.0x1.0mm, F.Cu at (124.2, 51.5)
- added TP7: CS, TestPoint:TestPoint_Pad_1.0x1.0mm, F.Cu at (84.3, 22.9)
- added V_IN2: 5V, TerminalBlock:TerminalBlock_Altech_AK300-2_P5.00mm, F.Cu at (109.1, 34.8)
- D6: value SS34-E3_57T -> SS34; footprint Diode_SMD:DIOM7959X262N -> Diode_SMD:D_SMC
- moved D6 0.24 mm to (53.1, 51.3), turned to 0 degrees
Connections:
- J1 pad 23: +5V -> 5V_OPI
- J1 pad 25: +5V -> 5V_OPI
- J2 pad 1: +5V -> 5V_OPI
- V_IN1 pad 2: Net-(V_IN1-Pin_2) -> +5V
Routing:
- net Net-(V_IN1-Pin_2): track 10.8 -> 0.00 mm
- net +5V: track 199.9 -> 210.7 mm
