File: Julelys.kicad_pcb (KiCad board)
At the start: 4 copper layers, 65 x 56 mm, 138 parts, among them J1 Raspberry_Pi_40pin, J10 B3B-XH-A, J11 B3B-XH-A, J12 Conn_01x03_Pin, J4 B3B-XH-A, J5 B3B-XH-A, J6 B3B-XH-A, J7 B3B-XH-A, J8 B3B-XH-A, J9 B3B-XH-A, P1 USB_C_Receptacle_USB2.0, SW1 SW_Push, SW2 SW_Push, U1 ESP32-C3FH4, U11 SRV05-4, U12 SRV05-4, U2 74HC4051, U3 AMS1117-3.3, U6 74AHCT1G125, U7 74AHCT1G125, U8 74AHCT1G125, U9 74AHCT1G125, Y1 40MHz

Commit message: Test board: read 8 analog sensors through the LED JST outputs
- U6 /OE now on IO1 (R51 10k pull-down keeps it on at boot); IO1 high
  tri-states the LED data shifter.
- /Data -> R52 15k -> IO0 (ADC1_CH0) -> R53 10k + C40 10nF to GND, so the
  mux can route any JST data pin back to the ADC (0-5 V -> 0-2 V).
- Placed and routed; references re-placed. 0 DRC errors, 0 unconnected,
  no silkscreen warnings, ERC unchanged.
- docs/sensor-input.md: how it works, read sequence, limits.

Co-Authored-By: Claude Opus 5.5 <noreply@anthropic.com>
Parts:
- added C40: 10nF, Capacitor_SMD:C_0402_1005Metric, F.Cu at (63.4, 36.0)
- added R51: 10k, Resistor_SMD:R_0402_1005Metric, F.Cu at (66.2, 37.9)
- added R52: 15k, Resistor_SMD:R_0402_1005Metric, F.Cu at (58.9, 41.5)
- added R53: 10k, Resistor_SMD:R_0402_1005Metric, F.Cu at (66.9, 34.0)
Connections:
- U6 pad 1: GND -> IO1
Routing:
- net IO0: track 7.52 -> 46.2 mm, vias 2 -> 10
- net IO1: track 9.90 -> 46.9 mm, vias 2 -> 3
- net /Data: track 16.1 -> 26.2 mm, vias 2 -> 3
- net GND: track 182.0 -> 183.8 mm, vias 221 -> 223

Commit message: R42 -> 510R (C25123) and D4 -> B5819W (C8598), both JLC Basic parts
Saves two extended-part setup fees. Same footprints; JLC rotation and
polarity checked (CPL unchanged).

Co-Authored-By: Claude Opus 5.5 <noreply@anthropic.com>
Parts:
- D4: value 1N5819HW-7-F -> B5819W
- R42: value 499 -> 510
Changed lines of the file:
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@@
 			)
 		)
-		(property "Value" "1N5819HW-7-F"
+		(property "Value" "B5819W"
 			(at 0 2.1 90)
 			(layer "F.Fab")
@@
 			)
 		)
-		(property "Value" "499"
+		(property "Value" "510"
 			(at 0 1.17 180)
 			(layer "F.Fab")
