File: power.kicad_sch (KiCad schematic)
At the start: 13 parts, among them SW1 SW_Push, SW2 SW_Push, U3 AMS1117-3.3

Commit message: version 3
Parts:
- added R12, R13: 10k, Resistor_SMD:R_0402_1005Metric, symbol Device:R
- added U4: BC847BDW1T1G, Transistor_Power_Module:SOT65P210X110-6N, symbol Transistor_Array:BC847BDW1T1G
- C4, C5, C6, C7: footprint Capacitor_SMD:C_0805_2012Metric -> Capacitor_SMD:C_0603_1608Metric
- H1, H2, H3, H4: footprint MountingHole:MountingHole_3mm -> MountingHole:MountingHole_3.2mm_M3
- R5: footprint Resistor_SMD:R_0805_2012Metric -> Resistor_SMD:R_0603_1608Metric
Connections:
- net CHIP_UP: now also U4.6 (COLLECTOR2)
- net IO9: now also U4.3 (COLLECTOR1)
- new net: R13.2, U4.2 (BASE2)
- new net: R12.1, U4.5 (BASE1)
- new net DTR: R12.2, U4.1 (EMITTER2)
- new net RTS: R13.1, U4.4 (EMITTER1)

Commit message: Update to v3.1
Parts:
- R12, R13: footprint Resistor_SMD:R_0402_1005Metric -> Resistor_SMD:R_0603_1608Metric
Changed lines of the file:
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@@
       (effects (font (size 1.27 1.27)))
     )
-    (property "Footprint" "Resistor_SMD:R_0402_1005Metric" (at 171.45 131.318 90)
+    (property "Footprint" "Resistor_SMD:R_0603_1608Metric" (at 171.45 131.318 90)
       (effects (font (size 1.27 1.27)) hide)
     )
@@
       (effects (font (size 1.27 1.27)))
     )
-    (property "Footprint" "Resistor_SMD:R_0402_1005Metric" (at 254 131.318 90)
+    (property "Footprint" "Resistor_SMD:R_0603_1608Metric" (at 254 131.318 90)
       (effects (font (size 1.27 1.27)) hide)
     )

Commit message: Begin next step
Parts:
- added C8: 470uF, Capacitor_SMD:CP_Elec_8x10, symbol Device:C_Polarized_US
- added C9: 100nF, Capacitor_SMD:C_0603_1608Metric, symbol Device:C
- added D6: SS34, Diode_SMD:D_SMC, symbol Device:D_Schottky
- added TP3: 3.3V, TestPoint:TestPoint_Pad_1.0x1.0mm, symbol Connector:TestPoint
Connections:
- net +3.3V: now also TP3.1
- net +5V: now also D6.1 (K)
- net GND: now also C8.2, C9.2
- new net 5V_OPI: C8.1, C9.1, D6.2 (A)
Other:
- note added: "Orange Pi Power Protection 5V -> Diode -> Capacitor -> Orange Pi Prevents LED current from draining OPi supply"

Commit message: more to next step
Parts:
- removed R12, R13: 10k, Resistor_SMD:R_0603_1608Metric, symbol Device:R
- removed U4: BC847BDW1T1G, Transistor_Power_Module:SOT65P210X110-6N, symbol Transistor_Array:BC847BDW1T1G
- renumbered C8 to C15, C9 to C16
Changed lines of the file:
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@@
   (junction (at 77.47 111.76) (diameter 0) (color 0 0 0 0)
   )
-  (junction (at 270.51 111.76) (diameter 0) (color 0 0 0 0)
-  )
   (junction (at 87.63 55.88) (diameter 0) (color 0 0 0 0)
   )
@@
   (junction (at 63.5 41.91) (diameter 0) (color 0 0 0 0)
   )
-  (junction (at 157.48 129.54) (diameter 0) (color 0 0 0 0)
-  )
   (junction (at 77.47 86.36) (diameter 0) (color 0 0 0 0)
   )
@@
     (stroke (width 0) (type default))
   )
-  (wire (pts (xy 257.81 129.54) (xy 270.51 129.54))
-    (stroke (width 0) (type default))
-  )
   (wire (pts (xy 91.44 111.76) (xy 77.47 111.76))
     (stroke (width 0) (type default))
@@
     (stroke (width 0) (type default))
   )
-  (wire (pts (xy 168.91 132.08) (xy 180.34 132.08))
-    (stroke (width 0) (type default))
-  )
   (wire (pts (xy 114.3 86.36) (xy 120.65 86.36))
     (stroke (width 0) (type default))
   )
-  (wire (pts (xy 246.38 147.32) (xy 157.48 147.32))
-    (stroke (width 0) (type default))
-  )
   (wire (pts (xy 63.5 55.88) (xy 87.63 55.88))
     (stroke (width 0) (type default))
@@
     (stroke (width 0) (type default))
   )
-  (wire (pts (xy 246.38 116.84) (xy 246.38 127))
-    (stroke (width 0) (type default))
-  )
   (wire (pts (xy 93.98 123.19) (xy 77.47 123.19))
     (stroke (width 0) (type default))
@@
     (stroke (width 0) (type default))
   )
-  (wire (pts (xy 175.26 129.54) (xy 180.34 129.54))
-    (stroke (width 0) (type default))
-  )
   (wire (pts (xy 114.3 97.79) (xy 114.3 86.36))
     (stroke (width 0) (type default))
   )
-  (wire (pts (xy 270.51 96.52) (xy 270.51 111.76))
-    (stroke (width 0) (type default))
-  )
   (wire (pts (xy 63.5 48.26) (xy 63.5 41.91))
     (stroke (width 0) (type default))
   )
-  (wire (pts (xy 246.38 129.54) (xy 250.19 129.54))
-    (stroke (width 0) (type default))
-  )
   (wire (pts (xy 87.63 55.88) (xy 113.03 55.88))
     (stroke (width 0) (type default))
@@
     (stroke (width 0) (type default))
   )
-  (wire (pts (xy 180.34 111.76) (xy 180.34 127))
-    (stroke (width 0) (type default))
-  )
   (wire (pts (xy 113.03 41.91) (xy 120.65 41.91))
     (stroke (width 0) (type default))
   )
-  (wire (pts (xy 157.48 115.57) (xy 157.48 129.54))
-    (stroke (width 0) (type default))
-  )
-  (wire (pts (xy 246.38 132.08) (xy 246.38 147.32))
-    (stroke (width 0) (type default))
-  )
   (wire (pts (xy 93.98 97.79) (xy 77.47 97.79))
     (stroke (width 0) (type default))
@@
     (stroke (width 0) (type default))
   )
-  (wire (pts (xy 157.48 129.54) (xy 167.64 129.54))
-    (stroke (width 0) (type default))
-  )
   (wire (pts (xy 189.23 59.69) (xy 189.23 62.23))
     (stroke (width 0) (type default))
   )
-  (wire (pts (xy 157.48 147.32) (xy 157.48 129.54))
-    (stroke (width 0) (type default))
-  )
-  (wire (pts (xy 270.51 111.76) (xy 180.34 111.76))
-    (stroke (width 0) (type default))
-  )
   (wire (pts (xy 189.23 45.72) (xy 189.23 52.07))
-    (stroke (width 0) (type default))
-  )
-  (wire (pts (xy 270.51 129.54) (xy 270.51 111.76))
-    (stroke (width 0) (type default))
-  )
-  (wire (pts (xy 246.38 116.84) (xy 257.81 116.84))
     (stroke (width 0) (type default))
   )
@@
     )
   )
-  (global_label "CHIP_UP" (shape input) (at 257.81 116.84 0) (fields_autoplaced)
-    (effects (font (size 1.27 1.27)) (justify left))
-    (property "Intersheetrefs" "${INTERSHEET_REFS}" (at 268.8386 116.84 0)
-      (effects (font (size 1.27 1.27)) (justify left) hide)
-    )
-  )
-  (global_label "IO9" (shape input) (at 168.91 132.08 180) (fields_autoplaced)
-    (effects (font (size 1.27 1.27)) (justify right))
-    (property "Intersheetrefs" "${INTERSHEET_REFS}" (at 162.78 132.08 0)
-      (effects (font (size 1.27 1.27)) (justify right) hide)
-    )
-  )
-  (global_label "RTS" (shape input) (at 157.48 115.57 90) (fields_autoplaced)
-    (effects (font (size 1.27 1.27)) (justify left))
-    (property "Intersheetrefs" "${INTERSHEET_REFS}" (at 157.48 109.1377 90)
-      (effects (font (size 1.27 1.27)) (justify left) hide)
-    )
-  )
-  (global_label "DTR" (shape input) (at 270.51 96.52 90) (fields_autoplaced)
-    (effects (font (size 1.27 1.27)) (justify left))
-    (property "Intersheetrefs" "${INTERSHEET_REFS}" (at 270.51 90.0272 90)
-      (effects (font (size 1.27 1.27)) (justify left) hide)
-    )
-  )
   (global_label "5V_OPI" (shape output) (at 264.16 41.91 0) (fields_autoplaced)
     (effects (font (size 1.27 1.27)) (justify left))
@@
     )
   )
-  (symbol (lib_id "Device:R") (at 171.45 129.54 90) (unit 1)
-    (in_bom yes) (on_board yes) (dnp no) (fields_autoplaced)
-    (property "Reference" "R13" (at 171.45 123.19 90)
-      (effects (font (size 1.27 1.27)))
-    )
-    (property "Value" "10k" (at 171.45 125.73 90)
-      (effects (font (size 1.27 1.27)))
-    )
-    (property "Footprint" "Resistor_SMD:R_0603_1608Metric" (at 171.45 131.318 90)
-      (effects (font (size 1.27 1.27)) hide)
-    )
-    (property "Datasheet" "~" (at 171.45 129.54 0)
-      (effects (font (size 1.27 1.27)) hide)
-    )
-    (pin "2")
-    (pin "1")
-    (instances
-      (project "Julelys"
-        (path "/9ef41b73-8dcb-4021-8930-5b1db22eb182/75d2635a-f2eb-4079-86f3-082e38564c79"
-          (reference "R13") (unit 1)
-        )
-      )
-    )
-  )
   (symbol (lib_id "Device:C_Polarized_US") (at 113.03 52.07 0) (unit 1)
     (in_bom yes) (on_board yes) (dnp no) (fields_autoplaced)
@@
         (path "/9ef41b73-8dcb-4021-8930-5b1db22eb182/75d2635a-f2eb-4079-86f3-082e38564c79"
           (reference "C5") (unit 1)
-        )
-      )
-    )
-  )
-  (symbol (lib_id "Device:R") (at 254 129.54 90) (unit 1)
-    (in_bom yes) (on_board yes) (dnp no) (fields_autoplaced)
-    (property "Reference" "R12" (at 254 123.19 90)
-      (effects (font (size 1.27 1.27)))
-    )
-    (property "Value" "10k" (at 254 125.73 90)
-      (effects (font (size 1.27 1.27)))
-    )
-    (property "Footprint" "Resistor_SMD:R_0603_1608Metric" (at 254 131.318 90)
-      (effects (font (size 1.27 1.27)) hide)
-    )
-    (property "Datasheet" "~" (at 254 129.54 0)
-      (effects (font (size 1.27 1.27)) hide)
-    )
-    (pin "2")
-    (pin "1")
-    (instances
-      (project "Julelys"
-        (path "/9ef41b73-8dcb-4021-8930-5b1db22eb182/75d2635a-f2eb-4079-86f3-082e38564c79"
-          (reference "R12") (unit 1)
         )
       )
@@
   (symbol (lib_id "Device:C_Polarized_US") (at 243.84 49.53 0) (unit 1)
     (in_bom yes) (on_board yes) (dnp no) (fields_autoplaced)
-    (property "Reference" "C8" (at 247.65 48.26 0)
-      (effects (font (size 1.27 1.27)) (justify left))
-    )
-    (property "Value" "470uF" (at 247.65 50.8 0)
+    (property "Reference" "C15" (at 247.65 47.625 0)
+      (effects (font (size 1.27 1.27)) (justify left))
+    )
+    (property "Value" "470uF" (at 247.65 50.165 0)
       (effects (font (size 1.27 1.27)) (justify left))
     )
@@
       (project "Julelys"
         (path "/9ef41b73-8dcb-4021-8930-5b1db22eb182/75d2635a-f2eb-4079-86f3-082e38564c79"
-          (reference "C8") (unit 1)
+          (reference "C15") (unit 1)
         )
       )
@@
   (symbol (lib_id "Device:C") (at 254 49.53 0) (unit 1)
     (in_bom yes) (on_board yes) (dnp no) (fields_autoplaced)
-    (property "Reference" "C9" (at 257.81 48.26 0)
+    (property "Reference" "C16" (at 257.81 48.26 0)
       (effects (font (size 1.27 1.27)) (justify left))
     )
@@
       (project "Julelys"
         (path "/9ef41b73-8dcb-4021-8930-5b1db22eb182/75d2635a-f2eb-4079-86f3-082e38564c79"
-          (reference "C9") (unit 1)
+          (reference "C16") (unit 1)
         )
       )
@@
         )
       )
-    )
-  )
-  (symbol (lib_id "Transistor_Array:BC847BDW1T1G") (at 180.34 127 0) (unit 1)
-    (in_bom yes) (on_board yes) (dnp no) (fields_autoplaced)
-    (property "Reference" "U4" (at 213.36 116.84 0)
-      (effects (font (size 1.524 1.524)))
-    )
-    (property "Value" "BC847BDW1T1G" (at 213.36 119.38 0)
-      (effects (font (size 1.524 1.524)))
-    )
-    (property "Footprint" "Transistor_Power_Module:SOT65P210X110-6N" (at 180.34 127 0)
-      (effects (font (size 1.27 1.27) italic) hide)
-    )
-    (property "Datasheet" "BC847BDW1T1G" (at 180.34 127 0)
-      (effects (font (size 1.27 1.27) italic) hide)
-    )
-    (pin "2")
-    (pin "1")
-    (pin "6")
-    (pin "5")
-    (pin "3")
-    (pin "4")
-    (instances
-      (project "Julelys"
-        (path "/9ef41b73-8dcb-4021-8930-5b1db22eb182/75d2635a-f2eb-4079-86f3-082e38564c79"
-          (reference "U4") (unit 1)
-        )
-      )
