File: untitled.kicad_sch (KiCad schematic)
At the start: 18 parts, among them J1 Conn_02x13_Top_Bottom, J12 Conn_01x03_Pin, J2 Conn_01x13, J3 Conn_02x06_Odd_Even, P1 USB_C_Receptacle_USB2.0, U5 CP2102N-A02-GQFN28

Commit message: Begin next step
Connections:
- net +5V: no longer J1.23 (Pin_23), J1.25 (Pin_25), J2.1 (Pin_1)
- new net 5V_OPI: J1.23 (Pin_23), J1.25 (Pin_25), J2.1 (Pin_1)
Changed lines of the file:
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@@
     (stroke (width 0) (type default))
   )
-  (wire (pts (xy 276.86 77.47) (xy 276.86 83.82))
+  (wire (pts (xy 276.86 88.9) (xy 276.86 83.82))
     (stroke (width 0) (type default))
   )
@@
     )
   )
+  (global_label "5V_OPI" (shape input) (at 276.86 88.9 270) (fields_autoplaced)
+    (effects (font (size 1.27 1.27)) (justify right))
+    (property "Intersheetrefs" "${INTERSHEET_REFS}" (at 276.86 96.0286 270)
+      (effects (font (size 1.27 1.27)) (justify right) hide)
+    )
+  )
   (global_label "DTR" (shape input) (at 135.89 143.51 0) (fields_autoplaced)
     (effects (font (size 1.27 1.27)) (justify left))
@@
     )
   )
+  (global_label "5V_OPI" (shape input) (at 186.69 96.52 0) (fields_autoplaced)
+    (effects (font (size 1.27 1.27)) (justify left))
+    (property "Intersheetrefs" "${INTERSHEET_REFS}" (at 196.1462 96.52 0)
+      (effects (font (size 1.27 1.27)) (justify left) hide)
+    )
+  )
   (global_label "CS" (shape input) (at 241.3 66.04 180) (fields_autoplaced)
     (effects (font (size 1.27 1.27)) (justify right))
@@
     (pin "1")
     (instances
-      (project "Julelys V2"
+      (project "Julelys"
         (path "/9ef41b73-8dcb-4021-8930-5b1db22eb182/1969c3e8-6100-4b45-a4c4-adbf98ab0c9d"
           (reference "#PWR018") (unit 1)
@@
     (pin "16")
     (instances
-      (project "Julelys V2"
+      (project "Julelys"
         (path "/9ef41b73-8dcb-4021-8930-5b1db22eb182/1969c3e8-6100-4b45-a4c4-adbf98ab0c9d"
           (reference "U5") (unit 1)
@@
     (pin "1")
     (instances
-      (project "Julelys V2"
+      (project "Julelys"
         (path "/9ef41b73-8dcb-4021-8930-5b1db22eb182/1969c3e8-6100-4b45-a4c4-adbf98ab0c9d"
           (reference "J2") (unit 1)
@@
     (pin "2")
     (instances
-      (project "Julelys V2"
+      (project "Julelys"
         (path "/9ef41b73-8dcb-4021-8930-5b1db22eb182/1969c3e8-6100-4b45-a4c4-adbf98ab0c9d"
           (reference "C9") (unit 1)
@@
     (pin "1")
     (instances
-      (project "Julelys V2"
+      (project "Julelys"
         (path "/9ef41b73-8dcb-4021-8930-5b1db22eb182/1969c3e8-6100-4b45-a4c4-adbf98ab0c9d"
           (reference "#PWR012") (unit 1)
@@
     )
   )
-  (symbol (lib_id "power:+5V") (at 276.86 77.47 0) (unit 1)
-    (in_bom yes) (on_board yes) (dnp no) (fields_autoplaced)
-    (property "Reference" "#PWR027" (at 276.86 81.28 0)
-      (effects (font (size 1.27 1.27)) hide)
-    )
-    (property "Value" "+5V" (at 276.86 72.39 0)
-      (effects (font (size 1.27 1.27)))
-    )
-    (property "Footprint" "" (at 276.86 77.47 0)
-      (effects (font (size 1.27 1.27)) hide)
-    )
-    (property "Datasheet" "" (at 276.86 77.47 0)
-      (effects (font (size 1.27 1.27)) hide)
-    )
-    (pin "1")
-    (instances
-      (project "Julelys V2"
-        (path "/9ef41b73-8dcb-4021-8930-5b1db22eb182/1969c3e8-6100-4b45-a4c4-adbf98ab0c9d"
-          (reference "#PWR027") (unit 1)
-        )
-      )
-    )
-  )
   (symbol (lib_id "Device:D") (at 72.39 52.07 180) (unit 1)
     (in_bom yes) (on_board yes) (dnp no) (fields_autoplaced)
@@
     (pin "2")
     (instances
-      (project "Julelys V2"
+      (project "Julelys"
         (path "/9ef41b73-8dcb-4021-8930-5b1db22eb182/1969c3e8-6100-4b45-a4c4-adbf98ab0c9d"
           (reference "D4") (unit 1)
@@
     (pin "1")
     (instances
-      (project "Julelys V2"
+      (project "Julelys"
         (path "/9ef41b73-8dcb-4021-8930-5b1db22eb182/1969c3e8-6100-4b45-a4c4-adbf98ab0c9d"
           (reference "R7") (unit 1)
@@
     (pin "1")
     (instances
-      (project "Julelys V2"
+      (project "Julelys"
         (path "/9ef41b73-8dcb-4021-8930-5b1db22eb182/1969c3e8-6100-4b45-a4c4-adbf98ab0c9d"
           (reference "R8") (unit 1)
@@
     (pin "1")
     (instances
-      (project "Julelys V2"
+      (project "Julelys"
         (path "/9ef41b73-8dcb-4021-8930-5b1db22eb182/1969c3e8-6100-4b45-a4c4-adbf98ab0c9d"
           (reference "#PWR019") (unit 1)
@@
     (pin "1")
     (instances
-      (project "Julelys V2"
+      (project "Julelys"
         (path "/9ef41b73-8dcb-4021-8930-5b1db22eb182/1969c3e8-6100-4b45-a4c4-adbf98ab0c9d"
           (reference "R24") (unit 1)
@@
     (pin "1")
     (instances
-      (project "Julelys V2"
+      (project "Julelys"
         (path "/9ef41b73-8dcb-4021-8930-5b1db22eb182/1969c3e8-6100-4b45-a4c4-adbf98ab0c9d"
           (reference "#PWR010") (unit 1)
@@
     (pin "1")
     (instances
-      (project "Julelys V2"
+      (project "Julelys"
         (path "/9ef41b73-8dcb-4021-8930-5b1db22eb182/1969c3e8-6100-4b45-a4c4-adbf98ab0c9d"
           (reference "#PWR025") (unit 1)
@@
     (pin "1")
     (instances
-      (project "Julelys V2"
+      (project "Julelys"
         (path "/9ef41b73-8dcb-4021-8930-5b1db22eb182/1969c3e8-6100-4b45-a4c4-adbf98ab0c9d"
           (reference "#PWR030") (unit 1)
@@
     (pin "1")
     (instances
-      (project "Julelys V2"
+      (project "Julelys"
         (path "/9ef41b73-8dcb-4021-8930-5b1db22eb182/1969c3e8-6100-4b45-a4c4-adbf98ab0c9d"
           (reference "R25") (unit 1)
@@
     (pin "1")
     (instances
-      (project "Julelys V2"
+      (project "Julelys"
         (path "/9ef41b73-8dcb-4021-8930-5b1db22eb182/1969c3e8-6100-4b45-a4c4-adbf98ab0c9d"
           (reference "R22") (unit 1)
@@
     (pin "1")
     (instances
-      (project "Julelys V2"
+      (project "Julelys"
         (path "/9ef41b73-8dcb-4021-8930-5b1db22eb182/1969c3e8-6100-4b45-a4c4-adbf98ab0c9d"
           (reference "#PWR08") (unit 1)
@@
     (pin "1")
     (instances
-      (project "Julelys V2"
+      (project "Julelys"
         (path "/9ef41b73-8dcb-4021-8930-5b1db22eb182/1969c3e8-6100-4b45-a4c4-adbf98ab0c9d"
           (reference "#PWR029") (unit 1)
@@
     (pin "3")
     (instances
-      (project "Julelys V2"
+      (project "Julelys"
         (path "/9ef41b73-8dcb-4021-8930-5b1db22eb182/1969c3e8-6100-4b45-a4c4-adbf98ab0c9d"
           (reference "D7") (unit 1)
@@
     (pin "18")
     (instances
-      (project "Julelys V2"
+      (project "Julelys"
         (path "/9ef41b73-8dcb-4021-8930-5b1db22eb182/1969c3e8-6100-4b45-a4c4-adbf98ab0c9d"
           (reference "J1") (unit 1)
@@
     )
   )
-  (symbol (lib_id "power:+5V") (at 186.69 96.52 0) (unit 1)
-    (in_bom yes) (on_board yes) (dnp no) (fields_autoplaced)
-    (property "Reference" "#PWR028" (at 186.69 100.33 0)
-      (effects (font (size 1.27 1.27)) hide)
-    )
-    (property "Value" "+5V" (at 186.69 91.44 0)
-      (effects (font (size 1.27 1.27)))
-    )
-    (property "Footprint" "" (at 186.69 96.52 0)
-      (effects (font (size 1.27 1.27)) hide)
-    )
-    (property "Datasheet" "" (at 186.69 96.52 0)
-      (effects (font (size 1.27 1.27)) hide)
-    )
-    (pin "1")
-    (instances
-      (project "Julelys V2"
-        (path "/9ef41b73-8dcb-4021-8930-5b1db22eb182/1969c3e8-6100-4b45-a4c4-adbf98ab0c9d"
-          (reference "#PWR028") (unit 1)
-        )
-      )
-    )
-  )
   (symbol (lib_id "power:GND") (at 60.96 170.18 0) (unit 1)
     (in_bom yes) (on_board yes) (dnp no) (fields_autoplaced)
@@
     (pin "1")
     (instances
-      (project "Julelys V2"
+      (project "Julelys"
         (path "/9ef41b73-8dcb-4021-8930-5b1db22eb182/1969c3e8-6100-4b45-a4c4-adbf98ab0c9d"
           (reference "#PWR026") (unit 1)
@@
     (pin "1")
     (instances
-      (project "Julelys V2"
+      (project "Julelys"
         (path "/9ef41b73-8dcb-4021-8930-5b1db22eb182/1969c3e8-6100-4b45-a4c4-adbf98ab0c9d"
           (reference "C10") (unit 1)
@@
     (pin "2")
     (instances
-      (project "Julelys V2"
+      (project "Julelys"
         (path "/9ef41b73-8dcb-4021-8930-5b1db22eb182/1969c3e8-6100-4b45-a4c4-adbf98ab0c9d"
           (reference "R10") (unit 1)
@@
     (pin "B6")
     (instances
-      (project "Julelys V2"
+      (project "Julelys"
         (path "/9ef41b73-8dcb-4021-8930-5b1db22eb182/1969c3e8-6100-4b45-a4c4-adbf98ab0c9d"
           (reference "P1") (unit 1)
@@
     (pin "1")
     (instances
-      (project "Julelys V2"
+      (project "Julelys"
         (path "/9ef41b73-8dcb-4021-8930-5b1db22eb182/1969c3e8-6100-4b45-a4c4-adbf98ab0c9d"
           (reference "#PWR020") (unit 1)
@@
     (pin "3")
     (instances
-      (project "Julelys V2"
+      (project "Julelys"
         (path "/9ef41b73-8dcb-4021-8930-5b1db22eb182/1969c3e8-6100-4b45-a4c4-adbf98ab0c9d"
           (reference "J12") (unit 1)
@@
     (pin "2")
     (instances
-      (project "Julelys V2"
+      (project "Julelys"
         (path "/9ef41b73-8dcb-4021-8930-5b1db22eb182/1969c3e8-6100-4b45-a4c4-adbf98ab0c9d"
           (reference "J3") (unit 1)
@@
     (pin "1")
     (instances
-      (project "Julelys V2"
+      (project "Julelys"
         (path "/9ef41b73-8dcb-4021-8930-5b1db22eb182/1969c3e8-6100-4b45-a4c4-adbf98ab0c9d"
           (reference "R9") (unit 1)
@@
     (pin "1")
     (instances
-      (project "Julelys V2"
+      (project "Julelys"
         (path "/9ef41b73-8dcb-4021-8930-5b1db22eb182/1969c3e8-6100-4b45-a4c4-adbf98ab0c9d"
           (reference "#PWR024") (unit 1)
@@
     (pin "1")
     (instances
-      (project "Julelys V2"
+      (project "Julelys"
         (path "/9ef41b73-8dcb-4021-8930-5b1db22eb182/1969c3e8-6100-4b45-a4c4-adbf98ab0c9d"
           (reference "#PWR023") (unit 1)
@@
     (pin "1")
     (instances
-      (project "Julelys V2"
+      (project "Julelys"
         (path "/9ef41b73-8dcb-4021-8930-5b1db22eb182/1969c3e8-6100-4b45-a4c4-adbf98ab0c9d"
           (reference "#PWR022") (unit 1)
@@
     (pin "2")
     (instances
-      (project "Julelys V2"
+      (project "Julelys"
         (path "/9ef41b73-8dcb-4021-8930-5b1db22eb182/1969c3e8-6100-4b45-a4c4-adbf98ab0c9d"
           (reference "R11") (unit 1)

Commit message: more to next step
Parts:
- added R12, R13: 10k, Resistor_SMD:R_0603_1608Metric, symbol Device:R
- added U4: BC847BDW1T1G, Transistor_Power_Module:SOT65P210X110-6N, symbol Transistor_Array:BC847BDW1T1G
Connections:
- net DTR: now also R13.2, U4.1 (EMITTER2)
- net IO9: now also U4.3 (COLLECTOR1)
- net RTS: now also R12.1, U4.4 (EMITTER1)
- new net: R12.2, U4.2 (BASE2)
- new net: R13.1, U4.5 (BASE1)
- new net CHIP_UP: U4.6 (COLLECTOR2)
Other:
- moved on the sheet: J12, J2, J3, R24, R25
